Commit message: add localizer package back in and add base-link in properly
just rename chassis base link no need for new link

File: src/description/urdf/athena_drive.urdf.xacro (robot description, xacro)
@@ -26,4 +26,10 @@
   <!-- Contains description of drive -->
   <xacro:description/>
+  <xacro:imu_sensor parent="base_link" prefix="rover">
+    <origin xyz="0 0 0.2" rpy="0 0 0"/>
+  </xacro:imu_sensor>
+  <xacro:gps_sensor parent="base_link" prefix="rover">
+    <origin xyz="0 0 0.3" rpy="0 0 0"/>
+  </xacro:gps_sensor>
   <xacro:if value="$(arg use_mock_hardware)">
     <xacro:athena_drive_ros2_control

Commit message: removed test package, added node functionality, renamed to just localizer

File: src/description/urdf/athena_drive.urdf.xacro (robot description, xacro)
@@ -27,8 +27,8 @@
   <!-- Contains description of drive -->
   <xacro:description/>
-  <xacro:imu_sensor parent="base_link" prefix="rover">
+  <xacro:imu_sensor parent="base_link">
     <origin xyz="0 0 0.2" rpy="0 0 0"/>
   </xacro:imu_sensor>
-  <xacro:gps_sensor parent="base_link" prefix="rover">
+  <xacro:gps_sensor parent="base_link">
     <origin xyz="0 0 0.3" rpy="0 0 0"/>
   </xacro:gps_sensor>

File: src/description/urdf/gps.xacro (robot description, xacro)
@@ -1,11 +1,11 @@
 <?xml version="1.0"?>
 <robot xmlns:xacro="http://www.ros.org/wiki/xacro">
-    <xacro:macro name="gps_sensor" params="parent prefix *origin">
-        <joint name="${prefix}_gps_joint" type="fixed">
+    <xacro:macro name="gps_sensor" params="parent *origin">
+        <joint name="gnss_joint" type="fixed">
             <xacro:insert_block name="origin" />
             <parent link="${parent}" />
-            <child link="${prefix}_gps_link" />
+            <child link="gnss_link" />
         </joint>
-        <link name="${prefix}_gps_link">
+        <link name="gnss_link">
             <visual>
                 <geometry>
@@ -17,10 +17,10 @@
             </visual>
         </link>
-        <gazebo reference="${prefix}_gps_link">
-            <sensor name="${prefix}_navsat" type="navsat">
+        <gazebo reference="gnss_link">
+            <sensor name="navsat" type="navsat">
                 <always_on>true</always_on>
                 <update_rate>10</update_rate>
                 <topic>/gps/fix</topic>
-                <ign_frame_id>${prefix}_gps_link</ign_frame_id>
+                <ign_frame_id>gnss_link</ign_frame_id>
                 <plugin filename="ignition-gazebo-navsat-system" name="ignition::gazebo::systems::NavSat"/>
             </sensor>

File: src/description/urdf/imu.xacro (robot description, xacro)
@@ -1,11 +1,11 @@
 <?xml version="1.0"?>
 <robot xmlns:xacro="http://www.ros.org/wiki/xacro">
-    <xacro:macro name="imu_sensor" params="parent prefix *origin">
-        <joint name="${prefix}_imu_joint" type="fixed">
+    <xacro:macro name="imu_sensor" params="parent *origin">
+        <joint name="imu_joint" type="fixed">
             <xacro:insert_block name="origin" />
             <parent link="${parent}" />
-            <child link="${prefix}_imu_link" />
+            <child link="imu_link" />
         </joint>
-        <link name="${prefix}_imu_link">
+        <link name="imu_link">
             <visual>
                 <geometry>
@@ -17,10 +17,10 @@
             </visual>
         </link>
-        <gazebo reference="${prefix}_imu_link">
-            <sensor name="${prefix}_imu" type="imu">
+        <gazebo reference="imu_link">
+            <sensor name="imu" type="imu">
                 <always_on>true</always_on>
                 <update_rate>100</update_rate>
                 <topic>/imu</topic>
-                <ign_frame_id>${prefix}_imu_link</ign_frame_id>
+                <ign_frame_id>imu_link</ign_frame_id>
                 <plugin filename="libignition-gazebo-imu-system.so" name="ignition::gazebo::systems::Imu"/>
             </sensor>

Commit message: make more realistic

File: src/description/urdf/athena_drive.urdf.xacro (robot description, xacro)
@@ -28,8 +28,8 @@
   <xacro:description/>
   <xacro:imu_sensor parent="base_link">
-    <origin xyz="0 0 0.2" rpy="0 0 0"/>
+    <origin xyz="0 0 0.0" rpy="0 0 0"/>
   </xacro:imu_sensor>
   <xacro:gps_sensor parent="base_link">
-    <origin xyz="0 0 0.3" rpy="0 0 0"/>
+    <origin xyz="0 0 0.0" rpy="0 0 0"/>
   </xacro:gps_sensor>
   <xacro:ground_truth_odometry/>

File: src/description/urdf/gps.xacro (robot description, xacro)
@@ -20,5 +20,5 @@
             <sensor name="navsat" type="navsat">
                 <always_on>true</always_on>
-                <update_rate>10</update_rate>
+                <update_rate>50</update_rate>
                 <topic>/gps/fix</topic>
                 <ign_frame_id>gnss_link</ign_frame_id>

File: src/description/urdf/imu.xacro (robot description, xacro)
@@ -20,5 +20,5 @@
             <sensor name="imu" type="imu">
                 <always_on>true</always_on>
-                <update_rate>100</update_rate>
+                <update_rate>200</update_rate>
                 <topic>/imu</topic>
                 <ign_frame_id>imu_link</ign_frame_id>

Commit message: Add localizer package back in and add base-link in properly (#15)
* added dependencies script and requirements.txt

* add localizer package back in and add base-link in properly

just rename chassis base link no need for new link

* added geographic lib to dependencies.sh

* add parameters and proper imu and gps transforms for localizer

* add ground truth odometry

* fix world loading and sensors

* removed test package, added node functionality, renamed to just localizer

* make more realistic

* remove old .rviz file

File: src/description/urdf/athena_drive.urdf.xacro (robot description, xacro)
@@ -9,4 +9,5 @@
   <xacro:include filename="imu.xacro"/>
   <xacro:include filename="gps.xacro"/>
+  <xacro:include filename="ground_truth_odom.xacro"/>
   <!-- Load robot's macro with parameters -->
   <!-- set prefix if multiple robots are used -->
@@ -24,4 +25,11 @@
   <!-- Contains description of drive -->
   <xacro:description/>
+  <xacro:imu_sensor parent="base_link">
+    <origin xyz="0 0 0.0" rpy="0 0 0"/>
+  </xacro:imu_sensor>
+  <xacro:gps_sensor parent="base_link">
+    <origin xyz="0 0 0.0" rpy="0 0 0"/>
+  </xacro:gps_sensor>
+  <xacro:ground_truth_odometry/>
   <xacro:if value="$(arg use_sim)">
     <xacro:athena_drive_ros2_control

Commit message: idfk

File: src/description/urdf/athena_drive.urdf.xacro (robot description, xacro)
@@ -28,8 +28,8 @@
   <xacro:description/>
   <xacro:imu_sensor parent="base_link">
-    <origin xyz="0 0 0.0" rpy="0 0 0"/>
+    <origin xyz="0.775305042176281 -0.0692748019047986 -0.475175318827691" rpy="0 0 0"/>
   </xacro:imu_sensor>
   <xacro:gps_sensor parent="base_link">
-    <origin xyz="0 0 0.0" rpy="0 0 0"/>
+    <origin xyz="0.775305042176281 -0.0692748019047986 -0.475175318827691" rpy="0 0 0"/>
   </xacro:gps_sensor>
   <xacro:ground_truth_odometry/>

Commit message: something?

File: src/description/urdf/athena_drive.urdf.xacro (robot description, xacro)
@@ -28,5 +28,5 @@
   <xacro:description/>
   <xacro:imu_sensor parent="base_link">
-    <origin xyz="0.775305042176281 -0.0692748019047986 -0.475175318827691" rpy="0 0 0"/>
+    <origin xyz="0.775305042176281 -0.0692748019047986 -0.475175318827691" rpy="0 0 -${pi}"/>
   </xacro:imu_sensor>
   <xacro:gps_sensor parent="base_link">

Commit message: almost maybe

File: src/description/urdf/athena_drive.urdf.xacro (robot description, xacro)
@@ -27,11 +27,11 @@
   <!-- Contains description of drive -->
   <xacro:description/>
-  <xacro:imu_sensor parent="base_link">
-    <origin xyz="0.775305042176281 -0.0692748019047986 -0.475175318827691" rpy="0 0 -${pi}"/>
+  <xacro:imu_sensor parent="base_footprint">
+    <origin xyz="0.0 0.0 0.0" rpy="0 0 0"/>
   </xacro:imu_sensor>
-  <xacro:gps_sensor parent="base_link">
-    <origin xyz="0.775305042176281 -0.0692748019047986 -0.475175318827691" rpy="0 0 0"/>
+  <xacro:gps_sensor parent="base_footprint">
+    <origin xyz="0.0 0.0 0.0" rpy="0 0 0"/>
   </xacro:gps_sensor>
-  <xacro:ground_truth_odometry/>
+  <!--<xacro:ground_truth_odometry robot_base_frame="base_footprint"/>-->
   <xacro:if value="$(arg use_mock_hardware)">
     <xacro:athena_drive_ros2_control

File: src/description/urdf/athena_drive_description.urdf.xacro (robot description, xacro)
@@ -6,11 +6,6 @@
     <xacro:macro name="description">
         <link name="base_link">
-            <inertial>
-                <origin xyz="0.775305042176281 -0.0692748019047986 -0.475175318827691" rpy="0 0 0" />
-                <mass value="44.0454429414672" />
-                <inertia ixx="1.41725466889743" ixy="0.00803894609354262" ixz="-1.19304822311593E-17" iyy="1.33698338807128" iyz="1.62926079635059E-16" izz="2.58380655400253" />
-            </inertial>
-            <visual>
-                <origin xyz="0 0 0" rpy="0 0 0" />
+            <visual>
+                <origin xyz="-0.775305042176281 0.0692748019047986 0.475175318827691" rpy="0 0 -0.094743" />
                 <geometry>
                     <mesh filename="package://description/meshes/chassis_base_link.STL" />
@@ -21,5 +16,5 @@
             </visual>
             <collision>
-                <origin xyz="0 0 0" rpy="0 0 0" />
+                <origin xyz="-0.775305042176281 0.0692748019047986 0.475175318827691" rpy="0 0 -0.094743" />
                 <geometry>
                     <mesh filename="package://description/meshes/chassis_base_link.STL" />
@@ -50,5 +45,5 @@
         </link>
         <joint name="suspension_front_left_joint" type="fixed">
-            <origin xyz="0.61263 0.22146 -0.74592" rpy="1.5708 0 0.094743" />
+            <origin xyz="-.13 0.2355 -.26" rpy="1.5708 0 0" />
             <parent link="base_link" />
             <child link="suspension_front_left_link" />
@@ -284,5 +279,5 @@
         <link name="suspension_front_right_link">
             <inertial>
-                <origin xyz="0.0996575069633246 0.177857108210349 0.0120793884653498" rpy="0 0 0" />
+                <origin xyz="0.0 0.177857108210349 0.0120793884653498" rpy="0 0 0" />
                 <mass value="0.815137674139981" />
                 <inertia ixx="0.00362369286611303" ixy="2.10533763884314E-06" ixz="-1.88068045019413E-07" iyy="0.0343314249178962" iyz="-6.67186692298955E-08" izz="0.0378758255771416" />
@@ -305,5 +300,5 @@
         </link>
         <joint name="suspension_front_right_joint" type="fixed">
-            <origin xyz="0.66803 -0.36146 -0.74592" rpy="1.5708 0 0.094743" />
+            <origin xyz="-.13 -0.36146 -.26" rpy="1.5708 0 0" />
             <parent link="base_link" />
             <child link="suspension_front_right_link" />
@@ -362,5 +357,5 @@
         </link>
         <joint name="steer_fr_joint" type="revolute">
-            <origin xyz="0 0 0.059903" rpy="3.1416 0.094743 3.1416" />
+            <origin xyz="0 0 0.059903" rpy="3.1416 0.0 3.1416" />
             <parent link="swerve_mount_2_link" />
             <child link="steer_2_link" />
@@ -391,5 +386,5 @@
         </link>
         <joint name="wheel_bracket_2_joint" type="fixed">
-            <origin xyz="0.0225042151326936 -0.128534743589743 0.0550203250295025" rpy="0 0.0947430505373176 0" />
+            <origin xyz="0.0225042151326936 -0.128534743589743 0.0550203250295025" rpy="0 0.0 0" />
             <parent link="steer_2_link" />
             <child link="wheel_bracket_2_link" />
@@ -475,5 +470,5 @@
         </link>
         <joint name="steer_br_joint" type="revolute">
-            <origin xyz="0 0 0.0599025014000917" rpy="0 -0.0947430505373176 0" />
+            <origin xyz="0 0 0.0599025014000917" rpy="0 0.0 0" />
             <parent link="swerve_mount_3_link" />
             <child link="steer_3_link" />
@@ -504,5 +499,5 @@
         </link>
         <joint name="wheel_bracket_3_joint" type="fixed">
-            <origin xyz="-0.011719658421911 -0.128534743589743 0.0584684115770519" rpy="0 0.0947430505373176 0" />
+            <origin xyz="-0.011719658421911 -0.128534743589743 0.0584684115770519" rpy="0 0.0 0" />
             <parent link="steer_3_link" />
             <child link="wheel_bracket_3_link" />
@@ -537,4 +532,11 @@
             <axis xyz="0 0 1" />
         </joint>
+        <!-- Base footprint frame with inverted X and Y axes -->
+        <link name="base_footprint" />
+        <joint name="base_footprint_joint" type="fixed">
+            <origin xyz="0 0 0" rpy="0 0 3.14159265359" />
+            <parent link="base_footprint" />
+            <child link="base_link" />
+        </joint>
     </xacro:macro>
 </robot>

Commit message: Update description and simulation configurations

File: src/description/urdf/athena_drive.urdf.xacro (robot description, xacro)
@@ -27,11 +27,11 @@
   <!-- Contains description of drive -->
   <xacro:description/>
-  <xacro:imu_sensor parent="base_link">
-    <origin xyz="0 0 0.0" rpy="0 0 0"/>
+  <xacro:imu_sensor parent="base_footprint">
+    <origin xyz="0.0 0.0 0.0" rpy="0 0 0"/>
   </xacro:imu_sensor>
-  <xacro:gps_sensor parent="base_link">
-    <origin xyz="0 0 0.0" rpy="0 0 0"/>
+  <xacro:gps_sensor parent="base_footprint">
+    <origin xyz="0.0 0.0 0.0" rpy="0 0 0"/>
   </xacro:gps_sensor>
-  <xacro:ground_truth_odometry/>
+  <xacro:ground_truth_odometry robot_base_frame="base_footprint"/>
   <xacro:if value="$(arg use_mock_hardware)">
     <xacro:athena_drive_ros2_control

Commit message: Added depth camera to urdf (#23)
Co-authored-by: Mohammad Durrani <46766905+mdurrani808@users.noreply.github.com>

File: src/description/urdf/athena_drive.urdf.xacro (robot description, xacro)
@@ -10,4 +10,5 @@
   <xacro:include filename="gps.xacro"/>
   <xacro:include filename="ground_truth_odom.xacro"/>
+  <xacro:include filename="depth_camera.xacro"/>
   <!-- Load robot's macro with parameters -->
   <!-- set prefix if multiple robots are used -->
@@ -32,4 +33,7 @@
   </xacro:gps_sensor>
   <xacro:ground_truth_odometry/>
+  <xacro:depth_camera parent_link="base_link">
+      <origin xyz="0.75 0 -0.37" rpy="0 0 0"/>
+  </xacro:depth_camera>
   <xacro:if value="$(arg use_sim)">
     <xacro:athena_drive_ros2_control

Commit message: Added ground truth tf publisher, updated URDF to follow proper coordinate conventions (#26)
* Update description and simulation configurations

* removed old xacro file

File: src/description/urdf/athena_drive.urdf.xacro (robot description, xacro)
@@ -26,11 +26,11 @@
   <!-- Contains description of drive -->
   <xacro:description/>
-  <xacro:imu_sensor parent="base_link">
-    <origin xyz="0 0 0.0" rpy="0 0 0"/>
+  <xacro:imu_sensor parent="base_footprint">
+    <origin xyz="0.0 0.0 0.0" rpy="0 0 0"/>
   </xacro:imu_sensor>
-  <xacro:gps_sensor parent="base_link">
-    <origin xyz="0 0 0.0" rpy="0 0 0"/>
+  <xacro:gps_sensor parent="base_footprint">
+    <origin xyz="0.0 0.0 0.0" rpy="0 0 0"/>
   </xacro:gps_sensor>
-  <xacro:ground_truth_odometry/>
+  <xacro:ground_truth_odometry robot_base_frame="base_footprint"/>
   <xacro:depth_camera parent_link="base_link">
       <origin xyz="0.75 0 -0.37" rpy="0 0 0"/>

Commit message: Depth Camera Visualization  (#27)
* added depth camera to urdf

* added rqt visualization for depth camera

---------

Co-authored-by: Mohammad Durrani <46766905+mdurrani808@users.noreply.github.com>

File: src/description/urdf/athena_drive.urdf.xacro (robot description, xacro)
@@ -33,6 +33,6 @@
   </xacro:gps_sensor>
   <xacro:ground_truth_odometry robot_base_frame="base_footprint"/>
-  <xacro:depth_camera parent_link="base_link">
-      <origin xyz="0.75 0 -0.37" rpy="0 0 0"/>
+  <xacro:depth_camera parent="base_footprint">
+      <origin xyz="0.0 0.0 0.1" rpy="0 0 0"/>
   </xacro:depth_camera>
   <xacro:if value="$(arg use_sim)">

Commit message: obstacle detection in rviz

File: src/description/urdf/athena_drive.urdf.xacro (robot description, xacro)
@@ -40,5 +40,5 @@
   <xacro:ground_truth_odometry robot_base_frame="base_footprint"/>
   <xacro:depth_camera parent="base_footprint">
-      <origin xyz="0.0 0.0 0.1" rpy="0 0 0"/>
+      <origin xyz=".5 0.1 0.1" rpy="0 0 0"/>
   </xacro:depth_camera>
   <xacro:if value="$(arg use_mock_hardware)">

File: src/description/urdf/depth_camera.xacro (robot description, xacro)
@@ -26,5 +26,5 @@
     </joint>
     <joint name="depth_camera_optical_joint" type="fixed">
-      <origin xyz="0 0 0" rpy="${-pi/2} 0 ${-pi/2}"/>
+      <origin xyz="0 0 0" rpy="0 0 0"/>
       <parent link="depth_camera_link"/>
       <child link="depth_camera_optical_frame"/>
@@ -33,9 +33,10 @@
       <sensor name="depth_camera" type="depth">
         <always_on>1</always_on>
-        <update_rate>10</update_rate>
+        <update_rate>50</update_rate>
         <visualize>true</visualize>
         <topic>depth_camera</topic>
+        <ign_frame_id>depth_camera_optical_frame</ign_frame_id>
         <camera name="depth_camera">
-          <horizontal_fov>1.05</horizontal_fov>
+          <horizontal_fov>2.0944</horizontal_fov>
           <image>
             <width>640</width>
@@ -45,5 +46,5 @@
           <clip>
             <near>0.1</near>
-            <far>10.0</far>
+            <far>20.0</far>
           </clip>
           <depth_camera>
