Commit message: unify hardware abstraction under use_sim, complete urdf joint coverage, remove dead sim controllers config

File: src/description/urdf/athena_drive.urdf.xacro (robot description, xacro)
@@ -3,9 +3,6 @@
   <!-- Use this if parameters are set from the launch file, otherwise delete -->
   <xacro:arg name="prefix" default=""/>
-  <xacro:arg name="use_mock_hardware" default="false"/>
-  <xacro:arg name="mock_sensor_commands" default="false"/>
-  <xacro:arg name="sim_gazebo" default="true"/>
+  <xacro:arg name="use_sim" default="false"/>
   <xacro:arg name="simulation_controllers" default=""/>
-  <xacro:include filename="$(find description)/urdf/athena_drive/athena_drive_macro.xacro"/>
   <xacro:include filename="$(find description)/urdf/athena_drive/athena_drive_macro.ros2_control.xacro"/>
   <xacro:include filename="imu.xacro"/>
@@ -42,14 +39,12 @@
       <origin xyz=".5 0.1 0.1" rpy="0 0 0"/>
   </xacro:depth_camera>
-  <xacro:if value="$(arg use_mock_hardware)">
+  <xacro:if value="$(arg use_sim)">
     <xacro:athena_drive_ros2_control
     name="athena_drive"
     prefix="$(arg prefix)"
-    use_mock_hardware="$(arg use_mock_hardware)"
-    mock_sensor_commands="$(arg mock_sensor_commands)"
-    sim_gazebo="$(arg sim_gazebo)"
+    use_sim="true"
     simulation_controllers="$(arg simulation_controllers)"/>
   </xacro:if>
-  <xacro:unless value="$(arg use_mock_hardware)">
+  <xacro:unless value="$(arg use_sim)">
     <xacro:odrive_ros2_control name="odrive"/>
     <xacro:rmd_ros2_control name="rmd"/>

File: src/description/urdf/athena_drive/athena_drive_macro.ros2_control.xacro (robot description, xacro)
@@ -1,125 +1,96 @@
 <?xml version="1.0" encoding="UTF-8"?>
 <robot xmlns:xacro="http://wiki.ros.org/xacro">
-  <xacro:macro name="athena_drive_ros2_control" params="
+    <xacro:macro name="athena_drive_ros2_control" params="
                name
-               prefix
-               use_mock_hardware:=false
-               mock_sensor_commands:=false
-               sim_gazebo:=false
-               simulation_controllers"
-               >
-    <ros2_control name="${name}" type="system">
-  <hardware>
-    <xacro:if value="${sim_gazebo}">
-      <plugin>gz_ros2_control/GazeboSimSystem</plugin>
-    </xacro:if>
-    <xacro:if value="${use_mock_hardware and not sim_gazebo}">
-      <plugin>mock_components/GenericSystem</plugin>
-      <param name="mock_sensor_commands">${mock_sensor_commands}</param>
-    </xacro:if>
-    <xacro:unless value="${use_mock_hardware or sim_gazebo}">
-      <plugin>mock_components/GenericSystem</plugin>
-    </xacro:unless>
-  </hardware>
-  <joint name="${prefix}suspension_front_left_joint">
-    <command_interface name="position">
-      <param name="min">-1.0471975512</param>
-      <param name="max">1.0471975512</param>
-    </command_interface>
-    <state_interface name="position">
-      <param name="initial_value">0.0</param>
-    </state_interface>
-    <state_interface name="velocity"/>
-  </joint>
-  <joint name="${prefix}suspension_front_right_joint">
-    <command_interface name="position">
-      <param name="min">-1.0471975512</param>
-      <param name="max">1.0471975512</param>
-    </command_interface>
-    <state_interface name="position">
-      <param name="initial_value">0.0</param>
-    </state_interface>
-    <state_interface name="velocity"/>
-  </joint>
-  <joint name="${prefix}steer_fl_joint">
-    <command_interface name="position">
-      <param name="min">-0.78539816339</param>
-      <param name="max">0.78539816339</param>
-    </command_interface>
-    <state_interface name="position">
-      <param name="initial_value">0.0</param>
-    </state_interface>
-    <state_interface name="velocity"/>
-  </joint>
-  <joint name="${prefix}steer_fr_joint">
-    <command_interface name="position">
-      <param name="min">-0.78539816339</param>
-      <param name="max">0.78539816339</param>
-    </command_interface>
-    <state_interface name="position">
-      <param name="initial_value">0.0</param>
-    </state_interface>
-    <state_interface name="velocity"/>
-  </joint>
-  <joint name="${prefix}steer_br_joint">
-    <command_interface name="position">
-      <param name="min">0.78539816339</param>
-      <param name="max">-0.78539816339</param>
-    </command_interface>
-    <state_interface name="position">
-      <param name="initial_value">0.0</param>
-    </state_interface>
-    <state_interface name="velocity"/>
-  </joint>
-  <joint name="${prefix}steer_bl_joint">
-    <command_interface name="position">
-      <param name="min">-0.78539816339</param>
-      <param name="max">0.78539816339</param>
-    </command_interface>
-    <state_interface name="position">
-      <param name="initial_value">0.0</param>
-    </state_interface>
-    <state_interface name="velocity"/>
-  </joint>
-  <joint name="${prefix}propulsion_fl_joint">
-    <command_interface name="velocity"/>
-    <state_interface name="position">
-      <param name="initial_value">0.0</param>
-    </state_interface>
-    <state_interface name="velocity"/>
-  </joint>
-  <joint name="${prefix}propulsion_fr_joint">
-    <command_interface name="velocity"/>
-    <state_interface name="position">
-      <param name="initial_value">0.0</param>
-    </state_interface>
-    <state_interface name="velocity"/>
-  </joint>
-  <joint name="${prefix}propulsion_br_joint">
-    <state_interface name="position">
-      <param name="initial_value">0.0</param>
-    </state_interface>
-    <state_interface name="velocity"/>
-  </joint>
-  <joint name="${prefix}propulsion_bl_joint">
-    <state_interface name="position">
-      <param name="initial_value">0.0</param>
-    </state_interface>
-    <state_interface name="velocity"/>
-  </joint>
-</ros2_control>
-    <xacro:if value="$(arg sim_gazebo)">
-      <gazebo>
-        <plugin filename="gz_ros2_control-system" name="gz_ros2_control::GazeboSimROS2ControlPlugin">
-          <xacro:if value="${simulation_controllers != ''}">
-            <parameters>${simulation_controllers}</parameters>
-          </xacro:if>
-          <controller_manager_node_name>${prefix}controller_manager</controller_manager_node_name>
-          <ros>
-            <remapping>ackermann_steering_controller/tf_odometry:=/tf</remapping>
-          </ros>
-        </plugin>
-      </gazebo>
-    </xacro:if>
-  </xacro:macro>
+               prefix use_sim:=false
+               simulation_controllers">
+        <ros2_control name="${name}" type="system">
+            <hardware>
+                <xacro:if value="${use_sim}">
+                    <plugin>gz_ros2_control/GazeboSimSystem</plugin>
+                </xacro:if>
+                <xacro:unless value="${use_sim}">
+                    <plugin>mock_components/GenericSystem</plugin>
+                </xacro:unless>
+            </hardware>
+            <joint name="${prefix}steer_fl_joint">
+                <command_interface name="position">
+                    <param name="min">0</param>
+                    <param name="max">6.2832</param>
+                </command_interface>
+                <state_interface name="position">
+                    <param name="initial_value">0.0</param>
+                </state_interface>
+                <state_interface name="velocity"/>
+            </joint>
+            <joint name="${prefix}steer_fr_joint">
+                <command_interface name="position">
+                    <param name="min">0</param>
+                    <param name="max">6.2832</param>
+                </command_interface>
+                <state_interface name="position">
+                    <param name="initial_value">0.0</param>
+                </state_interface>
+                <state_interface name="velocity"/>
+            </joint>
+            <joint name="${prefix}steer_br_joint">
+                <command_interface name="position">
+                    <param name="min">0</param>
+                    <param name="max">6.28318530718</param>
+                </command_interface>
+                <state_interface name="position">
+                    <param name="initial_value">0.0</param>
+                </state_interface>
+                <state_interface name="velocity"/>
+            </joint>
+            <joint name="${prefix}steer_bl_joint">
+                <command_interface name="position">
+                    <param name="min">0</param>
+                    <param name="max">6.2832</param>
+                </command_interface>
+                <state_interface name="position">
+                    <param name="initial_value">0.0</param>
+                </state_interface>
+                <state_interface name="velocity"/>
+            </joint>
+            <joint name="${prefix}propulsion_fl_joint">
+                <command_interface name="velocity"/>
+                <state_interface name="position">
+                    <param name="initial_value">0.0</param>
+                </state_interface>
+                <state_interface name="velocity"/>
+            </joint>
+            <joint name="${prefix}propulsion_fr_joint">
+                <command_interface name="velocity"/>
+                <state_interface name="position">
+                    <param name="initial_value">0.0</param>
+                </state_interface>
+                <state_interface name="velocity"/>
+            </joint>
+            <joint name="${prefix}propulsion_br_joint">
+                <command_interface name="velocity"/>
+                <state_interface name="position">
+                    <param name="initial_value">0.0</param>
+                </state_interface>
+                <state_interface name="velocity"/>
+            </joint>
+            <joint name="${prefix}propulsion_bl_joint">
+                <command_interface name="velocity"/>
+                <state_interface name="position">
+                    <param name="initial_value">0.0</param>
+                </state_interface>
+                <state_interface name="velocity"/>
+            </joint>
+        </ros2_control>
+        <xacro:if value="${use_sim}">
+            <gazebo>
+                <plugin filename="gz_ros2_control-system" name="gz_ros2_control::GazeboSimROS2ControlPlugin">
+                    <xacro:if value="${simulation_controllers != ''}">
+                        <parameters>${simulation_controllers}</parameters>
+                    </xacro:if>
+                    <controller_manager_node_name>${prefix}controller_manager</controller_manager_node_name>
+                </plugin>
+            </gazebo>
+        </xacro:if>
+    </xacro:macro>
 </robot>

Commit message: make depth camera config match zed URDF / config

File: src/description/urdf/athena_drive.urdf.xacro (robot description, xacro)
@@ -12,5 +12,5 @@
   <xacro:include filename="gps.xacro"/>
   <xacro:include filename="ground_truth_odom.xacro"/>
-  <xacro:include filename="depth_camera.xacro"/>
+  <xacro:include filename="zed_camera.xacro"/>
   <!-- Load robot's macro with parameters -->
   <!-- set prefix if multiple robots are used -->
@@ -39,7 +39,7 @@
   </xacro:gps_sensor>
   <xacro:ground_truth_odometry robot_base_frame="base_footprint"/>
-  <xacro:depth_camera parent="base_footprint">
-      <origin xyz=".5 0.1 0.1" rpy="0 0 0"/>
-  </xacro:depth_camera>
+  <xacro:zed_camera_sensor parent="base_footprint" camera_name="zed" camera_model="zed2i" sim_gazebo="$(arg sim_gazebo)">
+    <origin xyz=".5 0.1 0.1" rpy="0 0 0"/>
+  </xacro:zed_camera_sensor>
   <xacro:if value="$(arg use_mock_hardware)">
     <xacro:athena_drive_ros2_control
