Commit message: zed fixes

File: src/description/urdf/athena_drive.urdf.xacro (robot description, xacro)
@@ -39,5 +39,5 @@
   </xacro:gps_sensor>
   <xacro:ground_truth_odometry robot_base_frame="base_footprint"/>
-  <xacro:zed_camera_sensor parent="base_footprint" camera_name="zed" camera_model="zed2i" sim_gazebo="$(arg sim_gazebo)">
+  <xacro:zed_camera_sensor parent="base_footprint" camera_name="zed" sim_gazebo="$(arg sim_gazebo)">
     <origin xyz=".5 0.1 0.1" rpy="0 0 0"/>
   </xacro:zed_camera_sensor>

File: src/description/urdf/zed_camera.xacro (robot description, xacro)
@@ -6,9 +6,8 @@
       parent       - parent link to attach the camera to
       camera_name  - camera name used for all link/joint/topic names (default: zed)
-      camera_model - ZED model: zed, zedm, zed2, zed2i, zedx, zedxm, ... (default: zed2i)
       sim_gazebo   - when true, adds a Gazebo depth sensor on the left camera frame (default: false)
       *origin      - transform from parent to the camera mounting screw point
   -->
-  <xacro:macro name="zed_camera_sensor" params="parent camera_name:=zed camera_model:=zed2i sim_gazebo:=false *origin">
+  <xacro:macro name="zed_camera_sensor" params="parent camera_name:=zed sim_gazebo:=false *origin">
     <joint name="${camera_name}_mount_joint" type="fixed">
       <xacro:insert_block name="origin"/>
@@ -16,5 +15,5 @@
       <child link="${camera_name}_camera_link"/>
     </joint>
-    <xacro:zed_camera name="${camera_name}" model="${camera_model}" enable_gnss="false">
+    <xacro:zed_camera name="${camera_name}" enable_gnss="false">
       <origin xyz="0 0 0" rpy="0 0 0"/>
     </xacro:zed_camera>
@@ -46,4 +45,23 @@
           </plugin>
         </sensor>
+        <sensor name="${camera_name}_rgb_sensor" type="camera">
+          <always_on>1</always_on>
+          <update_rate>15</update_rate>
+          <visualize>true</visualize>
+          <topic>${camera_name}/zed_node/left/image_rect_color</topic>
+          <ign_frame_id>${camera_name}_left_camera_frame_optical</ign_frame_id>
+          <camera name="${camera_name}_rgb">
+            <horizontal_fov>1.8151</horizontal_fov>
+            <image>
+              <width>672</width>
+              <height>376</height>
+              <format>RGB_INT8</format>
+            </image>
+            <clip>
+              <near>0.2</near>
+              <far>20.0</far>
+            </clip>
+          </camera>
+        </sensor>
       </gazebo>
     </xacro:if>

File: src/description/urdf/zed_macro_sim.urdf.xacro (robot description, xacro)
@@ -2,181 +2,57 @@
 <robot xmlns:xacro="http://wiki.ros.org/xacro">
   <xacro:property name="M_PI" value="3.1415926535897931" />
-  <xacro:macro name="zed_camera" params="name=zed model=zed enable_gnss=false custom_baseline=0 *gnss_origin">
-    <xacro:if value="${model == 'zed'}">
-      <xacro:property name="baseline"         value="0.12"  />
-      <xacro:property name="height"           value="0.03"  />
-      <xacro:property name="bottom_slope"     value="0.05"  />
-      <xacro:property name="screw_offset_x"   value="0.0"   />
-      <xacro:property name="screw_offset_z"   value="0.0"   />
-      <xacro:property name="optical_offset_x" value="-0.01" />
-      <xacro:property name="mono"             value="false" />
-      <xacro:property name="mat"              value="0.8 0.8 0.8 1.0" />
-    </xacro:if>
-    <xacro:if value="${model == 'zedm'}">
-      <xacro:property name="baseline"         value="0.063" />
-      <xacro:property name="height"           value="0.0265"/>
-      <xacro:property name="bottom_slope"     value="0.0"   />
-      <xacro:property name="screw_offset_x"   value="0.0"   />
-      <xacro:property name="screw_offset_z"   value="0.0"   />
-      <xacro:property name="optical_offset_x" value="0.0"   />
-      <xacro:property name="mono"             value="false" />
-      <xacro:property name="mat"              value="0 0 0 1.0" />
-    </xacro:if>
-    <xacro:if value="${model == 'zed2'}">
-      <xacro:property name="baseline"         value="0.12"  />
-      <xacro:property name="height"           value="0.03"  />
-      <xacro:property name="bottom_slope"     value="0.05"  />
-      <xacro:property name="screw_offset_x"   value="0.0"   />
-      <xacro:property name="screw_offset_z"   value="0.0"   />
-      <xacro:property name="optical_offset_x" value="-0.01" />
-      <xacro:property name="mono"             value="false" />
-      <xacro:property name="mat"              value="0.25 0.25 0.25 1.0" />
-    </xacro:if>
-    <xacro:if value="${model == 'zed2i'}">
-      <xacro:property name="baseline"         value="0.12"  />
-      <xacro:property name="height"           value="0.03"  />
-      <xacro:property name="bottom_slope"     value="0.0"   />
-      <xacro:property name="screw_offset_x"   value="-0.01" />
-      <xacro:property name="screw_offset_z"   value="0.0"   />
-      <xacro:property name="optical_offset_x" value="-0.01" />
-      <xacro:property name="mono"             value="false" />
-      <xacro:property name="mat"              value="0.25 0.25 0.25 1.0" />
-    </xacro:if>
-    <xacro:if value="${model == 'zedx'}">
-      <xacro:property name="baseline"         value="0.12"  />
-      <xacro:property name="height"           value="0.032" />
-      <xacro:property name="bottom_slope"     value="0.0"   />
-      <xacro:property name="screw_offset_x"   value="0.0"   />
-      <xacro:property name="screw_offset_z"   value="-0.016"/>
-      <xacro:property name="optical_offset_x" value="-0.01" />
-      <xacro:property name="mono"             value="false" />
-      <xacro:property name="mat"              value="0.25 0.25 0.25 1.0" />
-    </xacro:if>
-    <xacro:if value="${model == 'zedxm'}">
-      <xacro:property name="baseline"         value="0.05"  />
-      <xacro:property name="height"           value="0.032" />
-      <xacro:property name="bottom_slope"     value="0.0"   />
-      <xacro:property name="screw_offset_x"   value="0.0"   />
-      <xacro:property name="screw_offset_z"   value="-0.016"/>
-      <xacro:property name="optical_offset_x" value="-0.01" />
-      <xacro:property name="mono"             value="false" />
-      <xacro:property name="mat"              value="0.25 0.25 0.25 1.0" />
-    </xacro:if>
-    <xacro:if value="${model == 'virtual'}">
-      <xacro:property name="baseline"         value="${custom_baseline}" />
-      <xacro:property name="height"           value="0.031" />
-      <xacro:property name="bottom_slope"     value="0.0"   />
-      <xacro:property name="screw_offset_x"   value="0.00"  />
-      <xacro:property name="screw_offset_z"   value="-0.0155"/>
-      <xacro:property name="optical_offset_x" value="0.0"   />
-      <xacro:property name="mono"             value="false" />
-      <xacro:property name="mat"              value="0.25 0.25 0.25 1.0" />
-    </xacro:if>
+  <xacro:macro name="zed_camera" params="name=zed enable_gnss=false *gnss_origin">
+    <xacro:property name="baseline"         value="0.12"  />
+    <xacro:property name="height"           value="0.03"  />
+    <xacro:property name="screw_offset_x"   value="-0.01" />
+    <xacro:property name="optical_offset_x" value="-0.01" />
     <!-- Camera mounting point (the threaded screw hole in the bottom) -->
     <link name="${name}_camera_link" />
-    <!-- Camera Center — mesh sourced from description package (no zed_msgs needed) -->
     <link name="${name}_camera_center">
-      <xacro:unless value="${model == 'virtual'}">
-        <visual>
-          <origin xyz="${screw_offset_x} 0 ${screw_offset_z}" rpy="0 0 0"/>
-          <geometry>
-            <mesh filename="file://$(find description)/meshes/${model}.stl"/>
-          </geometry>
-          <material name="zed_mat">
-            <color rgba="${mat}"/>
-          </material>
-        </visual>
-        <collision>
-          <origin xyz="${screw_offset_x} 0 ${screw_offset_z}" rpy="0 0 0"/>
-          <geometry>
-            <mesh filename="file://$(find description)/meshes/${model}.stl"/>
-          </geometry>
-        </collision>
-      </xacro:unless>
+      <visual>
+        <origin xyz="${screw_offset_x} 0 0" rpy="0 0 0"/>
+        <geometry>
+          <mesh filename="file://$(find description)/meshes/zed2i.stl"/>
+        </geometry>
+        <material name="zed_mat">
+          <color rgba="0.25 0.25 0.25 1.0"/>
+        </material>
+      </visual>
+      <collision>
+        <origin xyz="${screw_offset_x} 0 0" rpy="0 0 0"/>
+        <geometry>
+          <mesh filename="file://$(find description)/meshes/zed2i.stl"/>
+        </geometry>
+      </collision>
     </link>
     <joint name="${name}_camera_center_joint" type="fixed">
       <parent link="${name}_camera_link"/>
       <child link="${name}_camera_center"/>
-      <origin xyz="0 0 ${height/2}" rpy="0 ${bottom_slope} 0" />
+      <origin xyz="0 0 ${height/2}" rpy="0 0 0" />
     </joint>
-    <xacro:unless value="${mono}">
-      <!-- Left Camera -->
-      <link name="${name}_left_camera_frame">
-        <xacro:if value="${model == 'virtual'}">
-          <visual>
-            <origin xyz="0 0 0" rpy="0 0 0"/>
-            <geometry>
-              <mesh filename="file://$(find description)/meshes/${model}.stl"/>
-            </geometry>
-            <material name="zed_mat">
-              <color rgba="${mat}"/>
-            </material>
-          </visual>
-          <collision>
-            <origin xyz="0 0 0" rpy="0 0 0"/>
-            <geometry>
-              <mesh filename="file://$(find description)/meshes/${model}.stl"/>
-            </geometry>
-          </collision>
-        </xacro:if>
-      </link>
-      <joint name="${name}_left_camera_joint" type="fixed">
-        <parent link="${name}_camera_center"/>
-        <child link="${name}_left_camera_frame"/>
-        <origin xyz="${optical_offset_x} ${baseline/2} 0" rpy="0 0 0" />
-      </joint>
-      <link name="${name}_left_camera_frame_optical"/>
-      <joint name="${name}_left_camera_optical_joint" type="fixed">
-        <origin xyz="0 0 0" rpy="-${M_PI/2} 0.0 -${M_PI/2}"/>
-        <parent link="${name}_left_camera_frame"/>
-        <child link="${name}_left_camera_frame_optical"/>
-      </joint>
-      <!-- Right Camera -->
-      <link name="${name}_right_camera_frame">
-        <xacro:if value="${model == 'virtual'}">
-          <visual>
-            <origin xyz="0 0 0" rpy="0 0 0"/>
-            <geometry>
-              <mesh filename="file://$(find description)/meshes/${model}.stl"/>
-            </geometry>
-            <material name="zed_mat">
-              <color rgba="${mat}"/>
-            </material>
-          </visual>
-          <collision>
-            <origin xyz="0 0 0" rpy="0 0 0"/>
-            <geometry>
-              <mesh filename="file://$(find description)/meshes/${model}.stl"/>
-            </geometry>
-          </collision>
-        </xacro:if>
-      </link>
-      <joint name="${name}_right_camera_joint" type="fixed">
-        <parent link="${name}_camera_center"/>
-        <child link="${name}_right_camera_frame"/>
-        <origin xyz="${optical_offset_x} -${baseline/2} 0" rpy="0 0 0" />
-      </joint>
-      <link name="${name}_right_camera_frame_optical"/>
-      <joint name="${name}_right_camera_optical_joint" type="fixed">
-        <origin xyz="0 0 0" rpy="-${M_PI/2} 0.0 -${M_PI/2}"/>
-        <parent link="${name}_right_camera_frame"/>
-        <child link="${name}_right_camera_frame_optical"/>
-      </joint>
-    </xacro:unless>
-    <xacro:if value="${mono}">
-      <!-- Camera -->
-      <link name="${name}_camera_frame" />
-      <joint name="${name}_camera_joint" type="fixed">
-        <parent link="${name}_camera_center"/>
-        <child link="${name}_camera_frame"/>
-        <origin xyz="${optical_offset_x} 0 0" rpy="0 0 0" />
-      </joint>
-      <link name="${name}_camera_frame_optical"/>
-      <joint name="${name}_camera_optical_joint" type="fixed">
-        <origin xyz="0 0 0" rpy="-${M_PI/2} 0.0 -${M_PI/2}"/>
-        <parent link="${name}_camera_frame"/>
-        <child link="${name}_camera_frame_optical"/>
-      </joint>
-    </xacro:if>
+    <link name="${name}_left_camera_frame" />
+    <joint name="${name}_left_camera_joint" type="fixed">
+      <parent link="${name}_camera_center"/>
+      <child link="${name}_left_camera_frame"/>
+      <origin xyz="${optical_offset_x} ${baseline/2} 0" rpy="0 0 0" />
+    </joint>
+    <link name="${name}_left_camera_frame_optical"/>
+    <joint name="${name}_left_camera_optical_joint" type="fixed">
+      <origin xyz="0 0 0" rpy="-${M_PI/2} 0.0 -${M_PI/2}"/>
+      <parent link="${name}_left_camera_frame"/>
+      <child link="${name}_left_camera_frame_optical"/>
+    </joint>
+    <link name="${name}_right_camera_frame" />
+    <joint name="${name}_right_camera_joint" type="fixed">
+      <parent link="${name}_camera_center"/>
+      <child link="${name}_right_camera_frame"/>
+      <origin xyz="${optical_offset_x} -${baseline/2} 0" rpy="0 0 0" />
+    </joint>
+    <link name="${name}_right_camera_frame_optical"/>
+    <joint name="${name}_right_camera_optical_joint" type="fixed">
+      <origin xyz="0 0 0" rpy="-${M_PI/2} 0.0 -${M_PI/2}"/>
+      <parent link="${name}_right_camera_frame"/>
+      <child link="${name}_right_camera_frame_optical"/>
+    </joint>
     <xacro:if value="${enable_gnss}">
       <link name="${name}_gnss_link" />

Commit message: maybe fix the zed issue

File: src/description/urdf/athena_drive.urdf.xacro (robot description, xacro)
@@ -12,5 +12,4 @@
   <xacro:include filename="gps.xacro"/>
   <xacro:include filename="ground_truth_odom.xacro"/>
-  <xacro:include filename="zed_camera.xacro"/>
   <!-- Load robot's macro with parameters -->
   <!-- set prefix if multiple robots are used -->
@@ -39,7 +38,4 @@
   </xacro:gps_sensor>
   <xacro:ground_truth_odometry robot_base_frame="base_footprint"/>
-  <xacro:zed_camera_sensor parent="base_footprint" camera_name="zed" sim_gazebo="$(arg sim_gazebo)">
-    <origin xyz=".5 0.1 0.1" rpy="0 0 0"/>
-  </xacro:zed_camera_sensor>
   <xacro:if value="$(arg use_mock_hardware)">
     <xacro:athena_drive_ros2_control

Commit message: updated drive urdf

File: src/description/urdf/athena_drive.urdf.xacro (robot description, xacro)
@@ -12,4 +12,7 @@
   <xacro:include filename="gps.xacro"/>
   <xacro:include filename="ground_truth_odom.xacro"/>
+  <xacro:if value="$(arg sim_gazebo)">
+    <xacro:include filename="zed_camera.xacro"/>
+  </xacro:if>
   <!-- Load robot's macro with parameters -->
   <!-- set prefix if multiple robots are used -->
@@ -38,4 +41,9 @@
   </xacro:gps_sensor>
   <xacro:ground_truth_odometry robot_base_frame="base_footprint"/>
+  <xacro:if value="$(arg sim_gazebo)">
+    <xacro:zed_camera_sensor parent="base_footprint" camera_name="zed" sim_gazebo="$(arg sim_gazebo)">
+      <origin xyz=".5 0.1 0.1" rpy="0 0 0"/>
+    </xacro:zed_camera_sensor>
+  </xacro:if>
   <xacro:if value="$(arg use_mock_hardware)">
     <xacro:athena_drive_ros2_control

Commit message: Revert ZED-related changes from nav_testing_2324
Restores upstream/main versions of:
- sensors.launch.py (publish_odom/map defaults, gps_launch)
- zed.launch.py (publish_tf/publish_map_tf back to LaunchConfiguration)
- zed_macro_sim.urdf.xacro (color + rgb_sensor link/joint)
- athena_drive.urdf.xacro (unconditional zed include + original origin)
- nav_bringup.launch.py (remove zed_to_base_footprint static tf)

File: src/description/urdf/athena_drive.urdf.xacro (robot description, xacro)
@@ -12,7 +12,5 @@
   <xacro:include filename="gps.xacro"/>
   <xacro:include filename="ground_truth_odom.xacro"/>
-  <xacro:if value="$(arg sim_gazebo)">
-    <xacro:include filename="zed_camera.xacro"/>
-  </xacro:if>
+  <xacro:include filename="zed_camera.xacro"/>
   <!-- Load robot's macro with parameters -->
   <!-- set prefix if multiple robots are used -->
@@ -41,9 +39,7 @@
   </xacro:gps_sensor>
   <xacro:ground_truth_odometry robot_base_frame="base_footprint"/>
-  <xacro:if value="$(arg sim_gazebo)">
-    <xacro:zed_camera_sensor parent="base_footprint" camera_name="zed" sim_gazebo="$(arg sim_gazebo)">
-      <origin xyz=".5 0.1 0.1" rpy="0 0 0"/>
-    </xacro:zed_camera_sensor>
-  </xacro:if>
+  <xacro:zed_camera_sensor parent="base_footprint" camera_name="zed" sim_gazebo="$(arg sim_gazebo)">
+    <origin xyz=".3 -0.123 0.073" rpy="0 0 0"/>
+  </xacro:zed_camera_sensor>
   <xacro:if value="$(arg use_mock_hardware)">
     <xacro:athena_drive_ros2_control

File: src/description/urdf/zed_macro_sim.urdf.xacro (robot description, xacro)
@@ -16,5 +16,5 @@
         </geometry>
         <material name="zed_mat">
-          <color rgba="0.25 0.25 0.25 1.0"/>
+          <color rgba="0.08 0.08 0.08 1.0"/>
         </material>
       </visual>
@@ -43,4 +43,10 @@
       <child link="${name}_left_camera_frame_optical"/>
     </joint>
+    <link name="athena/base_footprint/${name}_rgb_sensor"/>
+    <joint name="${name}_rgb_sensor_joint" type="fixed">
+      <origin xyz="0 0 0" rpy="-${M_PI/2} 0.0 -${M_PI/2}"/>
+      <parent link="${name}_left_camera_frame"/>
+      <child link="athena/base_footprint/${name}_rgb_sensor"/>
+    </joint>
     <link name="${name}_right_camera_frame" />
     <joint name="${name}_right_camera_joint" type="fixed">

Commit message: building

File: src/description/urdf/athena_drive.urdf.xacro (robot description, xacro)
@@ -13,4 +13,5 @@
   <xacro:include filename="imu.xacro"/>
   <xacro:include filename="gps.xacro"/>
+  <xacro:include filename="magnetometer.xacro"/>
   <xacro:include filename="ground_truth_odom.xacro"/>
   <xacro:include filename="zed_camera.xacro"/>
@@ -40,4 +41,7 @@
     <origin xyz="0.0 0.0 0.0" rpy="0 0 0"/>
   </xacro:gps_sensor>
+  <xacro:magnetometer_sensor parent="base_footprint">
+    <origin xyz="0.0 0.0 0.0" rpy="0 0 0"/>
+  </xacro:magnetometer_sensor>
   <xacro:ground_truth_odometry robot_base_frame="base_footprint"/>
   <xacro:zed_camera_sensor parent="base_footprint" camera_name="zed" sim_gazebo="$(arg sim_gazebo)">

Commit message: building

File: src/description/urdf/athena_drive.urdf.xacro (robot description, xacro)
@@ -11,4 +11,5 @@
   <xacro:include filename="imu.xacro"/>
   <xacro:include filename="gps.xacro"/>
+  <xacro:include filename="magnetometer.xacro"/>
   <xacro:include filename="ground_truth_odom.xacro"/>
   <xacro:include filename="zed_camera.xacro"/>
@@ -38,4 +39,7 @@
     <origin xyz="0.0 0.0 0.0" rpy="0 0 0"/>
   </xacro:gps_sensor>
+  <xacro:magnetometer_sensor parent="base_footprint">
+    <origin xyz="0.0 0.0 0.0" rpy="0 0 0"/>
+  </xacro:magnetometer_sensor>
   <xacro:ground_truth_odometry robot_base_frame="base_footprint"/>
   <xacro:zed_camera_sensor parent="base_footprint" camera_name="zed" sim_gazebo="$(arg sim_gazebo)">
