Commit message: fix sim bringup

File: src/description/urdf/athena_drive/athena_drive_macro.ros2_control.xacro (robot description, xacro)
@@ -14,24 +14,4 @@
                 </xacro:unless>
             </hardware>
-            <joint name="${prefix}suspension_front_left_joint">
-                <command_interface name="position">
-                    <param name="min">-1.0471975512</param>
-                    <param name="max">1.0471975512</param>
-                </command_interface>
-                <state_interface name="position">
-                    <param name="initial_value">0.0</param>
-                </state_interface>
-                <state_interface name="velocity"/>
-            </joint>
-            <joint name="${prefix}suspension_front_right_joint">
-                <command_interface name="position">
-                    <param name="min">-1.0471975512</param>
-                    <param name="max">1.0471975512</param>
-                </command_interface>
-                <state_interface name="position">
-                    <param name="initial_value">0.0</param>
-                </state_interface>
-                <state_interface name="velocity"/>
-            </joint>
             <joint name="${prefix}steer_fl_joint">
                 <command_interface name="position">

Commit message: Nav Simulation Bringup Housecleaning (#29)
* **Package Dependency Fixes:**
- athena_map: Fix OpenCV dependency (opencv4 → libopencv-dev)
- athena_planner: Fix Nav2 planner dependency (nav2_planner_server → nav2_planner)
- obstacle_detection: Remove unused zed_interfaces dependency, fix PCL dependency (libpcl-dev → libpcl-all-dev)
- localizer: Add CMAKE_PREFIX_PATH for ROS2 GTSAM installation

* removed unused launch argument in gz_sim.launch.py

* [comments] Clarified world file origin

* updated spawn.launch.py to reflect convention

* Updated rear wheel joint names

* Changed rover name from 'rover' to 'athena'

* Added missing 'world_name' to ros_gz_sim create node params

* Changed IMU topic to unidirection (gazebo -> ros) from bidirectional

* Added velocity command interface to back propulsion joints

* Added simulation README.md for git lfs issue

* Added common issue and solution to simulation README.md

* added world_name param to sim spawn launch

* made ground_truth_tf_publisher executable

---------

Co-authored-by: Adrian Cires <loop@adriancires.com>

File: src/description/urdf/athena_drive/athena_drive_macro.ros2_control.xacro (robot description, xacro)
@@ -14,4 +14,24 @@
                 </xacro:unless>
             </hardware>
+            <joint name="${prefix}suspension_front_left_joint">
+                <command_interface name="position">
+                    <param name="min">-1.0471975512</param>
+                    <param name="max">1.0471975512</param>
+                </command_interface>
+                <state_interface name="position">
+                    <param name="initial_value">0.0</param>
+                </state_interface>
+                <state_interface name="velocity"/>
+            </joint>
+            <joint name="${prefix}suspension_front_right_joint">
+                <command_interface name="position">
+                    <param name="min">-1.0471975512</param>
+                    <param name="max">1.0471975512</param>
+                </command_interface>
+                <state_interface name="position">
+                    <param name="initial_value">0.0</param>
+                </state_interface>
+                <state_interface name="velocity"/>
+            </joint>
             <joint name="${prefix}steer_fl_joint">
                 <command_interface name="position">

Commit message: not really sure why this works but it works 4/7 times so

File: src/description/urdf/athena_drive/athena_drive_macro.ros2_control.xacro (robot description, xacro)
@@ -44,6 +44,6 @@
   <joint name="${prefix}steer_fl_joint">
     <command_interface name="position">
-      <param name="min">0</param>
-      <param name="max">6.2832</param>
+      <param name="min">-0.78539816339</param>
+      <param name="max">0.78539816339</param>
     </command_interface>
     <state_interface name="position">
@@ -54,6 +54,6 @@
   <joint name="${prefix}steer_fr_joint">
     <command_interface name="position">
-      <param name="min">0</param>
-      <param name="max">6.2832</param>
+      <param name="min">-0.78539816339</param>
+      <param name="max">0.78539816339</param>
     </command_interface>
     <state_interface name="position">
@@ -64,6 +64,6 @@
   <joint name="${prefix}steer_br_joint">
     <command_interface name="position">
-      <param name="min">0</param>
-      <param name="max">6.28318530718</param>
+      <param name="min">0.78539816339</param>
+      <param name="max">-0.78539816339</param>
     </command_interface>
     <state_interface name="position">
@@ -74,6 +74,6 @@
   <joint name="${prefix}steer_bl_joint">
     <command_interface name="position">
-      <param name="min">0</param>
-      <param name="max">6.2832</param>
+      <param name="min">-0.78539816339</param>
+      <param name="max">0.78539816339</param>
     </command_interface>
     <state_interface name="position">
@@ -97,5 +97,4 @@
   </joint>
   <joint name="${prefix}propulsion_br_joint">
-    <command_interface name="velocity"/>
     <state_interface name="position">
       <param name="initial_value">0.0</param>
@@ -104,5 +103,4 @@
   </joint>
   <joint name="${prefix}propulsion_bl_joint">
-    <command_interface name="velocity"/>
     <state_interface name="position">
       <param name="initial_value">0.0</param>

File: src/description/urdf/athena_drive_description.urdf.xacro (robot description, xacro)
@@ -106,5 +106,5 @@
             <child link="steer_1_link" />
             <axis xyz="0 1 0" />
-            <limit lower="-3.1416" upper="3.1416" effort="200" velocity="3" />
+            <limit lower="-0.78539816339" upper="0.78539816339" effort="200" velocity="3" />
         </joint>
         <link name="wheel_bracket_1_link">
@@ -219,5 +219,5 @@
             <child link="steer_4_link" />
             <axis xyz="0 1 0" />
-            <limit lower="-3.1416" upper="3.1416" effort="200" velocity="3" />
+            <limit lower="-0.78539816339" upper="0.78539816339" effort="200" velocity="3" />
         </joint>
         <link name="wheel_bracket_4_link">
@@ -361,5 +361,5 @@
             <child link="steer_2_link" />
             <axis xyz="0 1 0" />
-            <limit lower="-3.1416" upper="3.1416" effort="200" velocity="3" />
+            <limit lower="-0.78539816339" upper="0.78539816339" effort="200" velocity="3" />
         </joint>
         <link name="wheel_bracket_2_link">
@@ -474,5 +474,5 @@
             <child link="steer_3_link" />
             <axis xyz="0 1 0" />
-            <limit lower="-3.1416" upper="3.1416" effort="200" velocity="3" />
+            <limit lower="-0.78539816339" upper="0.78539816339" effort="200" velocity="3" />
         </joint>
         <link name="wheel_bracket_3_link">

Commit message: idfk

File: src/description/urdf/athena_drive/athena_drive_macro.ros2_control.xacro (robot description, xacro)
@@ -7,8 +7,8 @@
         <ros2_control name="${name}" type="system">
             <hardware>
-                <xacro:if value="$(arg use_sim)">
+                <xacro:if value="${use_sim}">
                     <plugin>gz_ros2_control/GazeboSimSystem</plugin>
                 </xacro:if>
-                <xacro:unless value="$(arg use_sim)">
+                <xacro:unless value="${use_sim}">
                     <plugin>mock_components/GenericSystem</plugin>
                 </xacro:unless>
@@ -83,5 +83,5 @@
             </joint>
         </ros2_control>
-        <xacro:if value="$(arg use_sim)">
+        <xacro:if value="${use_sim}">
             <gazebo>
                 <plugin filename="gz_ros2_control-system" name="gz_ros2_control::GazeboSimROS2ControlPlugin">

File: src/description/urdf/athena_drive/athena_drive_macro.xacro (robot description, xacro)
@@ -220,4 +220,107 @@
       <limit effort="0" lower="${radians(-360)}" upper="${radians(360)}" velocity="${radians(720)}"/>
     </joint>
+    <!-- Placeholder links/joints for the three missing wheels (steer_fr, steer_br, steer_bl,
+         propulsion_fr, propulsion_br).  These are simple cylinders so ros2_control can find
+         all 8 required joints when this macro is used directly. -->
+    <!-- link 7: front-right steer -->
+    <link name="${prefix}link7">
+      <xacro:default_inertial/>
+      <visual>
+        <origin xyz="0 0 0" rpy="0 0 0"/>
+        <geometry><cylinder length="0.3" radius="0.15"/></geometry>
+        <material name="blue"/>
+      </visual>
+      <collision>
+        <origin xyz="0 0 0" rpy="0 0 0"/>
+        <geometry><cylinder length="0.3" radius="0.15"/></geometry>
+      </collision>
+    </link>
+    <joint name="${prefix}steer_fr_joint" type="revolute">
+      <origin xyz="0 -0.6 0.3" rpy="${pi} 0 0"/>
+      <parent link="${prefix}base_link"/>
+      <child link="${prefix}link7"/>
+      <axis xyz="0 0 1"/>
+      <limit effort="0" lower="${radians(-180)}" upper="${radians(180)}" velocity="${radians(180)}"/>
+    </joint>
+    <!-- link 8: front-right propulsion -->
+    <link name="${prefix}link8">
+      <xacro:default_inertial/>
+      <visual>
+        <origin xyz="0 0 0" rpy="0 0 0"/>
+        <geometry><cylinder length="0.15" radius="0.1"/></geometry>
+        <material name="red"/>
+      </visual>
+      <collision>
+        <origin xyz="0 0 0" rpy="0 0 0"/>
+        <geometry><cylinder length="0.15" radius="0.1"/></geometry>
+      </collision>
+    </link>
+    <joint name="${prefix}propulsion_fr_joint" type="revolute">
+      <origin xyz="0.8 0 0" rpy="0 0 0"/>
+      <parent link="${prefix}link7"/>
+      <child link="${prefix}link8"/>
+      <axis xyz="0 0 1"/>
+      <limit effort="0" lower="${radians(-90)}" upper="${radians(180)}" velocity="${radians(270)}"/>
+    </joint>
+    <!-- link 9: back-right steer -->
+    <link name="${prefix}link9">
+      <xacro:default_inertial/>
+      <visual>
+        <origin xyz="0 0 0" rpy="0 0 0"/>
+        <geometry><cylinder length="0.3" radius="0.15"/></geometry>
+        <material name="grey"/>
+      </visual>
+      <collision>
+        <origin xyz="0 0 0" rpy="0 0 0"/>
+        <geometry><cylinder length="0.3" radius="0.15"/></geometry>
+      </collision>
+    </link>
+    <joint name="${prefix}steer_br_joint" type="revolute">
+      <origin xyz="0 -0.6 -0.3" rpy="${pi} 0 0"/>
+      <parent link="${prefix}base_link"/>
+      <child link="${prefix}link9"/>
+      <axis xyz="0 0 1"/>
+      <limit effort="0" lower="${radians(-180)}" upper="${radians(180)}" velocity="${radians(180)}"/>
+    </joint>
+    <!-- link 10: back-right propulsion -->
+    <link name="${prefix}link10">
+      <xacro:default_inertial/>
+      <visual>
+        <origin xyz="0 0 0" rpy="0 0 0"/>
+        <geometry><cylinder length="0.15" radius="0.1"/></geometry>
+        <material name="orange"/>
+      </visual>
+      <collision>
+        <origin xyz="0 0 0" rpy="0 0 0"/>
+        <geometry><cylinder length="0.15" radius="0.1"/></geometry>
+      </collision>
+    </link>
+    <joint name="${prefix}propulsion_br_joint" type="revolute">
+      <origin xyz="0 0 -0.15" rpy="0 ${pi/2} 0"/>
+      <parent link="${prefix}link9"/>
+      <child link="${prefix}link10"/>
+      <axis xyz="0 0 1"/>
+      <limit effort="0" lower="${radians(-120)}" upper="${radians(120)}" velocity="${radians(540)}"/>
+    </joint>
+    <!-- link 11: back-left steer -->
+    <link name="${prefix}link11">
+      <xacro:default_inertial/>
+      <visual>
+        <origin xyz="0 0 0" rpy="0 0 0"/>
+        <geometry><cylinder length="0.3" radius="0.15"/></geometry>
+        <material name="brown"/>
+      </visual>
+      <collision>
+        <origin xyz="0 0 0" rpy="0 0 0"/>
+        <geometry><cylinder length="0.3" radius="0.15"/></geometry>
+      </collision>
+    </link>
+    <joint name="${prefix}steer_bl_joint" type="revolute">
+      <origin xyz="0 0.6 -0.3" rpy="${pi} 0 0"/>
+      <parent link="${prefix}base_link"/>
+      <child link="${prefix}link11"/>
+      <axis xyz="0 0 1"/>
+      <limit effort="0" lower="${radians(-180)}" upper="${radians(180)}" velocity="${radians(180)}"/>
+    </joint>
     <!-- tool frame - fixed frame -->
     <joint name="${prefix}suspension_front_right_joint-tool0" type="fixed">

Commit message: replace use_mock_hardware/sim_gazebo with use_sim, fix steer_br limits, add velocity cmd to all propulsion joints, remove tf remapping

File: src/description/urdf/athena_drive/athena_drive_macro.ros2_control.xacro (robot description, xacro)
@@ -1,96 +1,118 @@
 <?xml version="1.0" encoding="UTF-8"?>
 <robot xmlns:xacro="http://wiki.ros.org/xacro">
-    <xacro:macro name="athena_drive_ros2_control" params="
+  <xacro:macro name="athena_drive_ros2_control" params="
                name
-               prefix use_sim:=false
-               simulation_controllers">
-        <ros2_control name="${name}" type="system">
-            <hardware>
-                <xacro:if value="${use_sim}">
-                    <plugin>gz_ros2_control/GazeboSimSystem</plugin>
-                </xacro:if>
-                <xacro:unless value="${use_sim}">
-                    <plugin>mock_components/GenericSystem</plugin>
-                </xacro:unless>
-            </hardware>
-            <joint name="${prefix}steer_fl_joint">
-                <command_interface name="position">
-                    <param name="min">0</param>
-                    <param name="max">6.2832</param>
-                </command_interface>
-                <state_interface name="position">
-                    <param name="initial_value">0.0</param>
-                </state_interface>
-                <state_interface name="velocity"/>
-            </joint>
-            <joint name="${prefix}steer_fr_joint">
-                <command_interface name="position">
-                    <param name="min">0</param>
-                    <param name="max">6.2832</param>
-                </command_interface>
-                <state_interface name="position">
-                    <param name="initial_value">0.0</param>
-                </state_interface>
-                <state_interface name="velocity"/>
-            </joint>
-            <joint name="${prefix}steer_br_joint">
-                <command_interface name="position">
-                    <param name="min">0</param>
-                    <param name="max">6.28318530718</param>
-                </command_interface>
-                <state_interface name="position">
-                    <param name="initial_value">0.0</param>
-                </state_interface>
-                <state_interface name="velocity"/>
-            </joint>
-            <joint name="${prefix}steer_bl_joint">
-                <command_interface name="position">
-                    <param name="min">0</param>
-                    <param name="max">6.2832</param>
-                </command_interface>
-                <state_interface name="position">
-                    <param name="initial_value">0.0</param>
-                </state_interface>
-                <state_interface name="velocity"/>
-            </joint>
-            <joint name="${prefix}propulsion_fl_joint">
-                <command_interface name="velocity"/>
-                <state_interface name="position">
-                    <param name="initial_value">0.0</param>
-                </state_interface>
-                <state_interface name="velocity"/>
-            </joint>
-            <joint name="${prefix}propulsion_fr_joint">
-                <command_interface name="velocity"/>
-                <state_interface name="position">
-                    <param name="initial_value">0.0</param>
-                </state_interface>
-                <state_interface name="velocity"/>
-            </joint>
-            <joint name="${prefix}propulsion_br_joint">
-                <command_interface name="velocity"/>
-                <state_interface name="position">
-                    <param name="initial_value">0.0</param>
-                </state_interface>
-                <state_interface name="velocity"/>
-            </joint>
-            <joint name="${prefix}propulsion_bl_joint">
-                <command_interface name="velocity"/>
-                <state_interface name="position">
-                    <param name="initial_value">0.0</param>
-                </state_interface>
-                <state_interface name="velocity"/>
-            </joint>
-        </ros2_control>
-        <xacro:if value="${use_sim}">
-            <gazebo>
-                <plugin filename="gz_ros2_control-system" name="gz_ros2_control::GazeboSimROS2ControlPlugin">
-                    <xacro:if value="${simulation_controllers != ''}">
-                        <parameters>${simulation_controllers}</parameters>
-                    </xacro:if>
-                    <controller_manager_node_name>${prefix}controller_manager</controller_manager_node_name>
-                </plugin>
-            </gazebo>
-        </xacro:if>
-    </xacro:macro>
+               prefix
+               use_sim:=false
+               simulation_controllers"
+               >
+    <ros2_control name="${name}" type="system">
+  <hardware>
+    <xacro:if value="${use_sim}">
+      <plugin>gz_ros2_control/GazeboSimSystem</plugin>
+    </xacro:if>
+    <xacro:unless value="${use_sim}">
+      <plugin>mock_components/GenericSystem</plugin>
+    </xacro:unless>
+  </hardware>
+  <joint name="${prefix}suspension_front_left_joint">
+    <command_interface name="position">
+      <param name="min">-1.0471975512</param>
+      <param name="max">1.0471975512</param>
+    </command_interface>
+    <state_interface name="position">
+      <param name="initial_value">0.0</param>
+    </state_interface>
+    <state_interface name="velocity"/>
+  </joint>
+  <joint name="${prefix}suspension_front_right_joint">
+    <command_interface name="position">
+      <param name="min">-1.0471975512</param>
+      <param name="max">1.0471975512</param>
+    </command_interface>
+    <state_interface name="position">
+      <param name="initial_value">0.0</param>
+    </state_interface>
+    <state_interface name="velocity"/>
+  </joint>
+  <joint name="${prefix}steer_fl_joint">
+    <command_interface name="position">
+      <param name="min">-0.78539816339</param>
+      <param name="max">0.78539816339</param>
+    </command_interface>
+    <state_interface name="position">
+      <param name="initial_value">0.0</param>
+    </state_interface>
+    <state_interface name="velocity"/>
+  </joint>
+  <joint name="${prefix}steer_fr_joint">
+    <command_interface name="position">
+      <param name="min">-0.78539816339</param>
+      <param name="max">0.78539816339</param>
+    </command_interface>
+    <state_interface name="position">
+      <param name="initial_value">0.0</param>
+    </state_interface>
+    <state_interface name="velocity"/>
+  </joint>
+  <joint name="${prefix}steer_br_joint">
+    <command_interface name="position">
+      <param name="min">-0.78539816339</param>
+      <param name="max">0.78539816339</param>
+    </command_interface>
+    <state_interface name="position">
+      <param name="initial_value">0.0</param>
+    </state_interface>
+    <state_interface name="velocity"/>
+  </joint>
+  <joint name="${prefix}steer_bl_joint">
+    <command_interface name="position">
+      <param name="min">-0.78539816339</param>
+      <param name="max">0.78539816339</param>
+    </command_interface>
+    <state_interface name="position">
+      <param name="initial_value">0.0</param>
+    </state_interface>
+    <state_interface name="velocity"/>
+  </joint>
+  <joint name="${prefix}propulsion_fl_joint">
+    <command_interface name="velocity"/>
+    <state_interface name="position">
+      <param name="initial_value">0.0</param>
+    </state_interface>
+    <state_interface name="velocity"/>
+  </joint>
+  <joint name="${prefix}propulsion_fr_joint">
+    <command_interface name="velocity"/>
+    <state_interface name="position">
+      <param name="initial_value">0.0</param>
+    </state_interface>
+    <state_interface name="velocity"/>
+  </joint>
+  <joint name="${prefix}propulsion_br_joint">
+    <command_interface name="velocity"/>
+    <state_interface name="position">
+      <param name="initial_value">0.0</param>
+    </state_interface>
+    <state_interface name="velocity"/>
+  </joint>
+  <joint name="${prefix}propulsion_bl_joint">
+    <command_interface name="velocity"/>
+    <state_interface name="position">
+      <param name="initial_value">0.0</param>
+    </state_interface>
+    <state_interface name="velocity"/>
+  </joint>
+</ros2_control>
+    <xacro:if value="${use_sim}">
+      <gazebo>
+        <plugin filename="gz_ros2_control-system" name="gz_ros2_control::GazeboSimROS2ControlPlugin">
+          <xacro:if value="${simulation_controllers != ''}">
+            <parameters>${simulation_controllers}</parameters>
+          </xacro:if>
+          <controller_manager_node_name>${prefix}controller_manager</controller_manager_node_name>
+        </plugin>
+      </gazebo>
+    </xacro:if>
+  </xacro:macro>
 </robot>
