Commit message: update rear ackermann controller

File: src/description/ros2_control/drive/drive.odrive.ros2_control.xacro (robot description, xacro)
@@ -27,4 +27,24 @@
         <state_interface name="velocity"/>
       </joint>
+      <joint name="steer_bl_joint">
+        <param name="node_id">TODO</param>
+        <param name="gear_ratio">26</param>
+        <command_interface name="position"/>
+        <command_interface name="velocity"/>
+        <state_interface name="position">
+          <param name="initial_value">0.0</param>
+        </state_interface>
+        <state_interface name="velocity"/>
+      </joint>
+      <joint name="steer_br_joint">
+        <param name="node_id">TODO</param>
+        <param name="gear_ratio">26</param>
+        <command_interface name="position"/>
+        <command_interface name="velocity"/>
+        <state_interface name="position">
+          <param name="initial_value">0.0</param>
+        </state_interface>
+        <state_interface name="velocity"/>
+      </joint>
     </ros2_control>
   </xacro:macro>

Commit message: remove todo nodes

File: src/description/ros2_control/drive/drive.odrive.ros2_control.xacro (robot description, xacro)
@@ -7,5 +7,5 @@
         <param name="can">can0</param>
       </hardware>
-      <joint name="steer_fl_joint">
+      <joint name="steer_bl_joint">
         <param name="node_id">5</param>
         <param name="gear_ratio">26</param>
@@ -17,26 +17,6 @@
         <state_interface name="velocity"/>
       </joint>
-      <joint name="steer_fr_joint">
+      <joint name="steer_br_joint">
         <param name="node_id">6</param>
-        <param name="gear_ratio">26</param>
-        <command_interface name="position"/>
-        <command_interface name="velocity"/>
-        <state_interface name="position">
-          <param name="initial_value">0.0</param>
-        </state_interface>
-        <state_interface name="velocity"/>
-      </joint>
-      <joint name="steer_bl_joint">
-        <param name="node_id">TODO</param>
-        <param name="gear_ratio">26</param>
-        <command_interface name="position"/>
-        <command_interface name="velocity"/>
-        <state_interface name="position">
-          <param name="initial_value">0.0</param>
-        </state_interface>
-        <state_interface name="velocity"/>
-      </joint>
-      <joint name="steer_br_joint">
-        <param name="node_id">TODO</param>
         <param name="gear_ratio">26</param>
         <command_interface name="position"/>
