Commit message: single launch file

File: src/description/ros2_control/arm/arm.rmd.ros2_control.xacro (robot description, xacro)
@@ -5,5 +5,5 @@
       <hardware>
         <plugin>rmd_ros2_control/RMDHardwareInterface</plugin>
-        <param name="update_rate">10</param> <!-- Hz -->
+        <param name="update_rate">2</param> <!-- Hz -->
         <param name="logger_rate">5</param> <!-- Hz -->
         <param name="logger_state">0</param> <!-- 0 for off, 1 for on -->
@@ -11,5 +11,5 @@
       </hardware>
       <joint name="shoulder_pitch">
-        <param name="node_id">0x14A</param>
+        <param name="node_id">0x149</param>
         <param name="gear_ratio">100</param>
         <param name="joint_orientation">1.0</param>

File: src/description/ros2_control/arm/arm.servo.ros2_control.xacro (robot description, xacro)
@@ -5,5 +5,5 @@
             <hardware>
                 <plugin>servo_ros2_control/SERVOHardwareInterface</plugin>
-                <param name="update_rate">10</param> <!-- Hz -->
+                <param name="update_rate">1</param> <!-- Hz -->
                 <param name="logger_rate">5</param> <!-- Hz -->
                 <param name="logger_state">0</param> <!-- 0 for off, 1 for on -->

File: src/description/ros2_control/arm/arm.smc.ros2_control.xacro (robot description, xacro)
@@ -5,5 +5,5 @@
       <hardware>
         <plugin>smc_ros2_control/SMCHardwareInterface</plugin>
-        <param name="update_rate">10</param> <!-- Hz -->
+        <param name="update_rate">2</param> <!-- Hz -->
         <param name="logger_rate">5</param> <!-- Hz -->
         <param name="logger_state">0</param> <!-- 0 for off, 1 for on -->
@@ -11,6 +11,6 @@
       </hardware>
       <joint name="base_yaw">
-        <param name="node_id">0x145</param>
-        <param name="gear_ratio">40</param>
+        <param name="node_id">0x148</param>
+        <param name="gear_ratio">-100</param>
         <param name="operating_velocity">300</param> <!-- motor dps -->
         <command_interface name="position"/>
@@ -22,5 +22,5 @@
       </joint>
       <joint name="wrist_pitch">
-        <param name="node_id">0x148</param>
+        <param name="node_id">0x145</param>
         <param name="gear_ratio">40</param>
         <param name="operating_velocity">1000</param> <!-- motor dps -->

File: src/description/ros2_control/drive/drive.rmd.ros2_control.xacro (robot description, xacro)
@@ -23,5 +23,5 @@
       </joint>
       <joint name="propulsion_fr_joint">
-        <param name="node_id">0x149</param>
+        <param name="node_id">0x150</param>
         <param name="gear_ratio">1</param>
         <param name="joint_orientation">1.0</param>

File: src/description/urdf/athena_arm.urdf.xacro (robot description, xacro)
@@ -32,5 +32,17 @@
   <xacro:unless value="$(arg use_mock_hardware)"> <!-- HARDWARE -->
     <xacro:smc_ros2_control name="smc"/>
-    <xacro:talon_ros2_control name="talon"/>
+    <ros2_control name="talon_mock" type="system">
+      <hardware>
+        <plugin>mock_components/GenericSystem</plugin>
+      </hardware>
+      <joint name="gripper_claw">
+        <command_interface name="position"/>
+        <command_interface name="velocity"/>
+        <state_interface name="position">
+          <param name="initial_value">-0.0</param>
+        </state_interface>
+        <state_interface name="velocity"/>
+      </joint>
+    </ros2_control>
     <xacro:rmd_ros2_control name="rmd"/>
     <xacro:servo_ros2_control name="servo"/>
